Commit message: spawn flyswatter on robot

File: src/drivers/universal_robot/ur_description/urdf/block.urdf (robot description, URDF)
Before this commit: robot block, 1 links, 0 joints
Links:
- link base_link: geometry collision box size=0.0318 0.0318 0.0318; visual mesh filename=package://ur_description/urdf/ur3/cockroach.dae scale=0.01 0.01 0.01

File: src/drivers/universal_robot/ur_description/urdf/ur3.urdf.xacro (robot description, xacro)
@@ -340,5 +340,6 @@
         <origin rpy="0 0 0" xyz="0 0 0"/>
         <geometry>
-          <cylinder radius="0.005" length="0.01"/>
+          <!-- <cylinder radius="0.005" length="0.01"/> -->
+          <mesh filename="package://ur_description/meshes/ur3/visual/flyswatter.dae" scale="0.01 0.01 0.01"/>
         </geometry>
       </visual>

Commit message: tried to load cockroach fialed

File: src/drivers/universal_robot/ur_description/urdf/block.urdf (robot description, URDF)
Before this commit: robot block, 1 links, 0 joints
Links:
- link base_link: geometry collision box size=0.0318 0.0318 0.0318; visual box size=0.0318 0.0318 0.0318

Commit message: tried and tried to load roachworld using roslaunch to no avail

File: src/drivers/universal_robot/ur_description/urdf/block.urdf (robot description, URDF)
Before this commit: robot block, 1 links, 0 joints
Links:
- link base_link: geometry collision box size=0.0318 0.0318 0.0318; visual mesh filename=package://ur_description/urdf/ur3/cockroach.dae scale=0.01 0.01 0.01
